Commit message: Maked subscription to wheelspeeds in teleop_to_serial and started implement transformations

File: ws/src/ground_drone_description/urdf/ground_drone.urdf.xacro (robot description, xacro)
@@ -2,5 +2,5 @@
 <robot xmlns:xacro="http://ros.org/wiki/xacro" name="ground_drone">
 <xacro:include filename="inertial_macros.xacro"/>
-  <link name="base_link">
+  <link name="base_footprint">
   </link>
   <!-- Define the main body -->
@@ -25,5 +25,5 @@
   </link>
   <joint name="body_to_base_link" type="fixed">
-    <parent link="base_link"/>
+    <parent link="base_footprint"/>
     <child link="body"/>
   </joint>
@@ -134,5 +134,5 @@
   <!-- Define joints -->
   <joint name="base_to_front_left_wheel" type="continuous">
-    <parent link="base_link"/>
+    <parent link="base_footprint"/>
     <child link="wheel_front_left"/>
     <origin xyz="0.5 -0.03 0" rpy="-1.5708 0 0"/>
@@ -140,5 +140,5 @@
   </joint>
   <joint name="base_to_front_right_wheel" type="continuous">
-    <parent link="base_link"/>
+    <parent link="base_footprint"/>
     <child link="wheel_front_right"/>
     <origin xyz="0.5 0.53 0" rpy="1.5708 0 0"/>
@@ -146,5 +146,5 @@
   </joint>
   <joint name="base_to_rear_left_wheel" type="continuous">
-    <parent link="base_link"/>
+    <parent link="base_footprint"/>
     <child link="wheel_rear_left"/>
     <origin xyz="0 -0.03 0" rpy="-1.5708 0 0"/>
@@ -152,5 +152,5 @@
   </joint>
   <joint name="base_to_rear_right_wheel" type="continuous">
-    <parent link="base_link"/>
+    <parent link="base_footprint"/>
     <child link="wheel_rear_right"/>
     <origin xyz="0 0.53 0" rpy="1.5708 0 0"/>
@@ -158,8 +158,7 @@
   </joint>
 <joint name="lidar_joint" type="fixed">
-    <parent link="base_link"/>
+    <parent link="base_footprint"/>
     <child link="lidar"/>
-    <origin xyz="0 0 0.1" rpy="0 0 0"/>
-    <limit effort="1" lower="-1.5708" upper="1.5708" velocity="1"/>
+    <origin xyz="0.25 0.25 0.25" rpy="0 0 0"/>
   </joint>
   <gazebo>
@@ -169,8 +168,8 @@
       <odometryFrame>odom</odometryFrame>
       <odometryRate>20.0</odometryRate>
-      <robotBaseFrame>body</robotBaseFrame>
+      <robotBaseFrame>base_footprint</robotBaseFrame>
       <wheel_radius>0.1</wheel_radius>
-      <base_length>0.651</base_length>
-      <base_width>0.246</base_width>
+      <base_length>0.430</base_length>
+      <base_width>0.315</base_width>
       <front_left_joint>base_to_front_left_wheel</front_left_joint>
       <front_right_joint>base_to_front_right_wheel</front_right_joint>
